Commit message: Allow for changing a custom sensor's joint rpy

File: urdf/utils/custom_sensors.xacro (robot description, xacro)
@@ -1,7 +1,8 @@
 <?xml version="1.0"?>
 <robot xmlns:xacro="https://www.ros.org/wiki/xacro">
-    <xacro:property name="side" value="foo"/>
+    <xacro:property name="id" value="foo"/>
     <xacro:property name="plink" value="foo_parent"/>
-    <xacro:property name="originjoint" value="foo_joint"/>
+    <xacro:property name="jointxyz" value="0 0 0"/>
+    <xacro:property name="jointrpy" value="0 0 0"/>
     <xacro:property name="sensor_width" value="0.007" />
     <xacro:property name="sensor_length" value="0.0025" />
@@ -9,6 +10,6 @@
     <xacro:property name="originrpy" value="0 0 0" />
     <xacro:property name="originxyz" value="0 0 0" />
-    <xacro:macro name="csensor" params="plink side mass originrpy originxyz originjoint">
-        <link name="sensor_${side}">
+    <xacro:macro name="csensor" params="plink id mass originrpy originxyz jointxyz jointrpy">
+        <link name="sensor_${id}">
             <visual>
                 <geometry>
@@ -27,11 +28,11 @@
                 <mass value="${mass}" />
                 <origin rpy="${originrpy}" xyz="${originxyz}" />
-                <box_inertia m="${mass}" x="${sensor_length}" y="${sensor_width}" z="${sensor_height}" />
+                <xacro:box_inertia mass="${mass}" x="${sensor_length}" y="${sensor_width}" z="${sensor_height}" />
             </inertial>
         </link>
-        <joint name="${plink}_sensor_${side}" type="fixed">
+        <joint name="${plink}_sensor_${id}" type="fixed">
             <parent link="${plink}" />
-            <child link="sensor_${side}" />
-            <origin xyz="${originjoint}" />
+            <child link="sensor_${id}" />
+            <origin xyz="${jointxyz}" rpy="${jointrpy}" />
         </joint>
     </xacro:macro>

Commit message: Fix thymio proximity sensor macro

File: urdf/utils/custom_sensors.xacro (robot description, xacro)
@@ -11,5 +11,5 @@
     <xacro:property name="originxyz" value="0 0 0" />
     <xacro:macro name="csensor" params="plink id mass originrpy originxyz jointxyz jointrpy">
-        <link name="sensor_${id}">
+        <link name="sensor_${id}_mount_point">
             <visual>
                 <geometry>
@@ -17,23 +17,83 @@
                 </geometry>
                 <material name="black" />
-                <origin rpy="${originrpy}" xyz="${originxyz}" />
+                <origin rpy="0 0 0" xyz="0 0 0" />
             </visual>
             <collision>
                 <geometry>
-                    <box size="${sensor_width} ${sensor_length} ${sensor_height}" />
+                    <box size="0 0 0" />
                 </geometry>
-                <origin rpy="${originrpy}" xyz="${originxyz}" />
+                <origin rpy="0 0 0" xyz="0 0 0" />
             </collision>
             <inertial>
                 <mass value="${mass}" />
-                <origin rpy="${originrpy}" xyz="${originxyz}" />
+                <origin rpy="0 0 0" xyz="0 0 0" />
+                <xacro:box_inertia mass="${mass}" x="${sensor_length}" y="${sensor_width}" z="${sensor_height}" />
+            </inertial>
+        </link>
+        <joint name="${plink}_sensor_${id}_mount_point" type="fixed">
+            <parent link="${plink}" />
+            <child link="sensor_${id}_mount_point" />
+            <origin xyz="${jointxyz}" rpy="${jointrpy}" />
+            <axis rpy="0 0 0" xyz="0 0 0"/>
+        </joint>
+        <link name="sensor_${id}">
+            <visual>
+                <geometry>
+                    <box size="0 0 0" />
+                </geometry>
+                <material name="black" />
+                <origin rpy="0 0 0" xyz="0 0 0" />
+            </visual>
+            <collision>
+                <geometry>
+                    <box size="0 0 0" />
+                </geometry>
+                <origin rpy="0 0 0" xyz="0 0 0" />
+            </collision>
+            <inertial>
+                <mass value="0" />
+                <origin rpy="0 0 0" xyz="0 0 0" />
                 <xacro:box_inertia mass="${mass}" x="${sensor_length}" y="${sensor_width}" z="${sensor_height}" />
             </inertial>
         </link>
         <joint name="${plink}_sensor_${id}" type="fixed">
-            <parent link="${plink}" />
+            <parent link="sensor_${id}_mount_point" />
             <child link="sensor_${id}" />
-            <origin xyz="${jointxyz}" rpy="${jointrpy}" />
+            <origin xyz="0 0 0" rpy="0 0 1.57" />
+            <axis rpy="0 0 0" xyz="0 0 0"/>
         </joint>
+        <gazebo reference="sensor_${id}">
+            <sensor type="ray" name="sensor_${id}_instance">
+                <pose>0 0 0 0 0 0</pose>
+                <ray>
+                    <scan>
+                        <horizontal>
+                            <samples>1</samples>
+                            <resolution>1</resolution>
+                            <min_angle>-0.05</min_angle>
+                            <max_angle>0.05</max_angle>
+                        </horizontal>
+                        <vertical>
+                            <samples>1</samples>
+                            <resolution>1</resolution>
+                            <min_angle>-0.05</min_angle>
+                            <max_angle>0.05</max_angle>
+                        </vertical>
+                    </scan>
+                    <range>
+                        <min>0.0005</min>
+                        <max>0.04</max>
+                        <resolution>0.0001</resolution>
+                    </range>
+                </ray>
+                <plugin name="laser" filename="libgazebo_ros_laser.so">
+                    <topicName>/thymio_laser/sensor_${id}</topicName>
+                    <frameName>sensor_${id}</frameName>
+                </plugin>
+                <always_on>true</always_on>
+                <update_rate>10</update_rate>
+                <visualize>true</visualize>
+            </sensor>
+        </gazebo>
     </xacro:macro>
 </robot>

Commit message: Added originrpy and originxyz.

File: urdf/utils/custom_sensors.xacro (robot description, xacro)
@@ -17,5 +17,5 @@
                 </geometry>
                 <material name="black" />
-                <origin rpy="0 0 0" xyz="0 0 0" />
+                <origin rpy="${originrpy}" xyz="${originxyz}" />
             </visual>
             <collision>
@@ -23,9 +23,9 @@
                     <box size="0 0 0" />
                 </geometry>
-                <origin rpy="0 0 0" xyz="0 0 0" />
+                <origin rpy="${originrpy}" xyz="${originxyz}" />
             </collision>
             <inertial>
                 <mass value="${mass}" />
-                <origin rpy="0 0 0" xyz="0 0 0" />
+                <origin rpy="${originrpy}" xyz="${originxyz}" />
                 <xacro:box_inertia mass="${mass}" x="${sensor_length}" y="${sensor_width}" z="${sensor_height}" />
             </inertial>
